Commit message: Adding SWIFT AUV

File: uuv_descriptions/urdf/rexrov_sensors.xacro (robot description, xacro)
@@ -23,5 +23,5 @@
     parent_link="${namespace}/base_link"
     inertial_reference_frame="${inertial_reference_frame}">
-    <origin xyz="-1.4 0 -0.312" rpy="0 ${0.5*pi} 0"/>
+    <origin xyz="-1.4 0 -0.321" rpy="0 ${0.5*pi} 0"/>
   </xacro:default_dvl_macro>
   <!-- Magnetometer  -->
@@ -33,5 +33,5 @@
   <!-- Pressure  -->
   <xacro:default_pressure_macro namespace="${namespace}" parent_link="${namespace}/base_link">
-    <origin xyz="-1.32 0.5 0.85" rpy="0 0 0"/>
+    <origin xyz="0 0.0 -0.7" rpy="0 0 0"/>
   </xacro:default_pressure_macro>
   <!-- IMU  -->
@@ -52,4 +52,8 @@
     <origin xyz="1.15 0.63 0.4" rpy="0 0.6 -0.4"/>
   </xacro:default_camera>
+    <!-- Forward-looking sonar sensor  -->
+  <xacro:forward_multibeam_p900 namespace="${namespace}" parent_link="${namespace}/base_link">
+    <origin xyz="1.4 0 0.65" rpy="0 0 0"/>
+  </xacro:forward_multibeam_p900> -->
   <!-- Mount a GPS. -->
   <xacro:default_gps namespace="${namespace}" parent_link="${namespace}/base_link" />

File: uuv_sensor_plugins/uuv_sensor_ros_plugins/urdf/camera_snippets.xacro (robot description, xacro)
@@ -33,5 +33,5 @@
       parent_link="${parent_link}"
       topic="camera"
-      mass="0.1"
+      mass="0.01"
       update_rate="30"
       hfov="1.5125"
@@ -39,5 +39,5 @@
       height="492"
       stddev="0.02"
-      scale="1.0">
+      scale="0.3">
       <inertia ixx="0.00001" ixy="0.0" ixz="0.0" iyy="0.00001" iyz="0.0" izz="0.00001" />
       <xacro:insert_block name="origin" />
@@ -56,5 +56,5 @@
       height="492"
       stddev="0.02"
-      scale="1.0">
+      scale="0.3">
       <inertia ixx="0.00001" ixy="0.0" ixz="0.0" iyy="0.00001" iyz="0.0" izz="0.00001" />
       <xacro:insert_block name="origin" />>

File: uuv_sensor_plugins/uuv_sensor_ros_plugins/urdf/dvl_snippets.xacro (robot description, xacro)
@@ -32,40 +32,40 @@
       parent_link="${parent_link}"
       reference_frame="${inertial_reference_frame}"
-      update_rate="7"
+      update_rate="15"
+      topic="dvl"
+      noise_sigma="0.01"
+      noise_amplitude="0"
+      scale="0.3">
+      <xacro:insert_block name="origin" />
+    </xacro:dvl_plugin_macro>
+  </xacro:macro>
+  <xacro:macro name="default_dvl_sensor_enu" params="namespace parent_link *origin">
+    <xacro:default_dvl_macro
+      namespace="${namespace}"
+      parent_link="${parent_link}"
+      reference_frame="world">
+      <xacro:insert_block name="origin" />
+    </xacro:default_dvl_macro>
+  </xacro:macro>
+  <xacro:macro name="default_dvl_sensor_ned" params="namespace parent_link *origin">
+    <xacro:default_dvl_macro
+      namespace="${namespace}"
+      parent_link="${parent_link}"
+      reference_frame="world_ned">
+      <xacro:insert_block name="origin" />
+    </xacro:default_dvl_macro>
+  </xacro:macro>
+  <!-- DEPRECATED MACRO: See default_dvl_sensor_enu -->
+  <xacro:macro name="default_dvl" params="namespace parent_link *origin">
+    <xacro:dvl_plugin_macro
+      namespace="${namespace}"
+      suffix=""
+      parent_link="${parent_link}"
+      reference_frame="world"
+      update_rate="15"
       topic="dvl"
       noise_sigma="0"
       noise_amplitude="0"
-      scale="1">
-      <xacro:insert_block name="origin" />
-    </xacro:dvl_plugin_macro>
-  </xacro:macro>
-  <xacro:macro name="default_dvl_sensor_enu" params="namespace parent_link *origin">
-    <xacro:default_dvl_macro
-      namespace="${namespace}"
-      parent_link="${parent_link}"
-      reference_frame="world">
-      <xacro:insert_block name="origin" />
-    </xacro:default_dvl_macro>
-  </xacro:macro>
-  <xacro:macro name="default_dvl_sensor_ned" params="namespace parent_link *origin">
-    <xacro:default_dvl_macro
-      namespace="${namespace}"
-      parent_link="${parent_link}"
-      reference_frame="world_ned">
-      <xacro:insert_block name="origin" />
-    </xacro:default_dvl_macro>
-  </xacro:macro>
-  <!-- DEPRECATED MACRO: See default_dvl_sensor_enu -->
-  <xacro:macro name="default_dvl" params="namespace parent_link *origin">
-    <xacro:dvl_plugin_macro
-      namespace="${namespace}"
-      suffix=""
-      parent_link="${parent_link}"
-      reference_frame="world"
-      update_rate="7"
-      topic="dvl"
-      noise_sigma="0"
-      noise_amplitude="0"
-      scale="1">
+      scale="0.3">
       <xacro:insert_block name="origin" />
     </xacro:dvl_plugin_macro>
@@ -109,5 +109,5 @@
           <range>
             <min>0.55</min>
-            <max>81</max>
+            <max>110</max>
             <resolution>0.01</resolution>
           </range>

File: uuv_sensor_plugins/uuv_sensor_ros_plugins/urdf/gps_sensor_snippets.xacro (robot description, xacro)
@@ -26,5 +26,5 @@
        <inertial>
          <inertia ixx="0.00001" ixy="0.0" ixz="0.0" iyy="0.00001" iyz="0.0" izz="0.00001" />
-         <mass value="${mass_gps_sensor}" />  <!-- [kg] -->
+         <mass value=".1" />  <!-- [kg] -->
          <origin xyz="0 0 0" rpy="0 0 0" />
        </inertial>

File: uuv_sensor_plugins/uuv_sensor_ros_plugins/urdf/imu_snippets.xacro (robot description, xacro)
@@ -42,6 +42,6 @@
       accelerometer_random_walk="0.006"
       accelerometer_bias_correlation_time="300.0"
-      accelerometer_turn_on_bias_sigma="0.1960"
-      orientation_noise="0.01"
+      accelerometer_turn_on_bias_sigma="0.01960"
+      orientation_noise="0.001"
       enable_local_ned_frame="false"
       reference_frame="world"
@@ -83,5 +83,5 @@
       accelerometer_random_walk="0.006"
       accelerometer_bias_correlation_time="300.0"
-      accelerometer_turn_on_bias_sigma="0.1960"
+      accelerometer_turn_on_bias_sigma="0.01960"
       orientation_noise="0.01"
       enable_local_ned_frame="false"
@@ -107,5 +107,5 @@
       accelerometer_random_walk="0.006"
       accelerometer_bias_correlation_time="300.0"
-      accelerometer_turn_on_bias_sigma="0.1960"
+      accelerometer_turn_on_bias_sigma="0.10960"
       orientation_noise="0.01"
       enable_local_ned_frame="true"

File: uuv_sensor_plugins/uuv_sensor_ros_plugins/urdf/pressure_snippets.xacro (robot description, xacro)
@@ -33,7 +33,7 @@
       topic="pressure"
       mass="0.015"
-      update_rate="10"
+      update_rate="20"
       range="30000"
-      noise_sigma="3.0"
+      noise_sigma="0.1"
       noise_amplitude="0.0"
       estimateDepth="false"
@@ -51,7 +51,7 @@
       topic="pressure"
       mass="0.015"
-      update_rate="10"
+      update_rate="20"
       range="30000"
-      noise_sigma="3.0"
+      noise_sigma="0.1"
       noise_amplitude="0.0"
       estimateDepth="false"
@@ -74,5 +74,5 @@
       <visual>
         <geometry>
-          <mesh filename="file://$(find uuv_sensor_ros_plugins)/meshes/pressure.dae" scale="1 1 1"/>
+          <mesh filename="file://$(find uuv_sensor_ros_plugins)/meshes/pressure.dae" scale="0.3 0.3 0.3"/>
         </geometry>
       </visual>

File: uuv_sensor_plugins/uuv_sensor_ros_plugins/urdf/rpt_snippets.xacro (robot description, xacro)
@@ -42,5 +42,5 @@
     <link name="${namespace}/rpt${suffix}_link">
       <inertial>
-        <mass value="0.001" />  <!-- [kg] -->
+        <mass value="2.25" />  <!-- [kg] -->
         <origin xyz="0 0 0" rpy="0 0 0" />
         <inertia ixx="0.000000017" ixy="0" ixz="0" iyy="0.000000017" iyz="0" izz="0.000000017" />

File: uuv_sensor_plugins/uuv_sensor_ros_plugins/urdf/sonar_snippets.xacro (robot description, xacro)
@@ -59,5 +59,5 @@
       parent_link="${parent_link}"
       topic="sonar"
-      mass="0.015"
+      mass="2.015"
       update_rate="25"
       samples="768"
@@ -94,5 +94,5 @@
       <visual>
         <geometry>
-          <mesh filename="file://$(find uuv_sensor_ros_plugins)/meshes/p900.dae" scale="1 1 1"/>
+          <mesh filename="file://$(find uuv_sensor_ros_plugins)/meshes/pingsonar.dae" scale="1 1 1"/>
         </geometry>
       </visual>
