Commit message: Simulator updates

File: swift_description/urdf/swift_actuators.xacro (robot description, xacro)
@@ -5,6 +5,6 @@
 <!-- Here you can put in whatever kind of model you want and it will
   still function as a propeller                                      -->
-  <xacro:property name="prop_mesh_file_cw" value="file://$(find swift_description)/mesh/t200_propccw.dae"/>
-  <xacro:property name="prop_mesh_file_ccw" value="file://$(find swift_description)/mesh/t200_propcw.dae"/>
+  <xacro:property name="prop_mesh_file_cw" value="file://$(find swift_description)/meshes/t200_propccw.dae"/>
+  <xacro:property name="prop_mesh_file_ccw" value="file://$(find swift_description)/meses/t200_propcw.dae"/>
   <!-- <xacro:property name="prop_mesh_file" value="file://$(find swift_description)/mesh/manipulator_claw.dae"/> -->
   <!-- Thruster joint and link snippet -->

File: swift_description/urdf/swift_base.xacro (robot description, xacro)
@@ -20,5 +20,5 @@
   -->
   <!-- Mass -->
-  <xacro:property name="mass" value="35.5"/>
+  <xacro:property name="mass" value="36.7"/>
   <!-- Describing the dimensions of the vehicle's bounding box: width, length, height -->
   <xacro:property name="x_size" value="0.74"/>
@@ -27,5 +27,5 @@
   <!-- minion_usv_height is not really! It's just for run... We need first calculate the Fossen parameters -->
   <!-- Volume -->
-  <xacro:property name="volume" value="0.0364"/>
+  <xacro:property name="volume" value="0.036"/>
   <!-- Center of gravity -->
   <!--xacro:property name="cog" value="0.0 0.0  0.0"/-->
@@ -46,5 +46,5 @@
   <!-- Parameters -->
   <xacro:property name="namespace" value="swift"/>
-  <xacro:property name="visual_mesh_file" value="file://$(find swift_description)/mesh/swift_body.stl"/>
+  <xacro:property name="visual_mesh_file" value="file://$(find swift_description)/meshes/swift_body.stl"/>
   <xacro:macro name="swift_base" params="namespace *gazebo inertial_reference_frame">
    <!-- Rigid body description of the base link -->

File: swift_description/urdf/swift_sensors.xacro (robot description, xacro)
@@ -21,4 +21,17 @@
   <!-- Magnetometer  -->
   <xacro:default_magnetometer namespace="${namespace}" parent_link="${namespace}/base_link"/>
+  <!-- Sonar  -->
+  <xacro:default_sonar_macro
+    namespace="${namespace}"
+    parent_link="${namespace}/base_link"
+    inertial_reference_frame="${inertial_reference_frame}">
+    <origin xyz="0.2 0 0.2125" rpy="0 0 0"/>
+  </xacro:default_sonar_macro>
+  <!-- Depth_Camera  -->
+  <xacro:zed2_macro
+    namespace="${namespace}"
+    parent_link="${namespace}/base_link">
+    <origin xyz="0.37 0.0 0.15" rpy="0 0 0"/>
+  </xacro:zed2_macro>
   <!-- Mount a Pose 3D sensor. This will give 3D pose -->
   <xacro:default_pose_3d_macro

File: uuv_descriptions/urdf/rexrov_sensors.xacro (robot description, xacro)
@@ -23,6 +23,19 @@
     parent_link="${namespace}/base_link"
     inertial_reference_frame="${inertial_reference_frame}">
-    <origin xyz="-1.4 0 -0.321" rpy="0 ${0.5*pi} 0"/>
+    <origin xyz="-1.44 0 -0.321" rpy="0 ${0.5*pi} 0"/>
   </xacro:default_dvl_macro>
+  <!-- Sonar  -->
+  <xacro:default_sonar_macro
+    namespace="${namespace}"
+    parent_link="${namespace}/base_link"
+    inertial_reference_frame="${inertial_reference_frame}">
+    <origin xyz="1.07 0 0.84" rpy="0 0 0"/>
+  </xacro:default_sonar_macro>
+  <!-- Depth_Camera  -->
+  <xacro:zed2_macro
+    namespace="${namespace}"
+    parent_link="${namespace}/base_link">
+    <origin xyz="1.3 0.0 0.6" rpy="0 0 0"/>
+  </xacro:zed2_macro>
   <!-- Magnetometer  -->
   <xacro:default_magnetometer namespace="${namespace}" parent_link="${namespace}/base_link"/>
@@ -42,18 +55,4 @@
     <origin xyz="0 0 0" rpy="0 0 0"/>
   </xacro:default_imu_macro>
-  <!-- Mount a camera -->
-  <xacro:default_camera namespace="${namespace}" parent_link="${namespace}/base_link" suffix="">
-    <origin xyz="1.15 0 0.4" rpy="0 0.6 0"/>
-  </xacro:default_camera>
-  <xacro:default_camera namespace="${namespace}" parent_link="${namespace}/base_link" suffix="right">
-    <origin xyz="1.15 -0.63 0.4" rpy="0 0.6 0.4"/>
-  </xacro:default_camera>
-  <xacro:default_camera namespace="${namespace}" parent_link="${namespace}/base_link" suffix="left">
-    <origin xyz="1.15 0.63 0.4" rpy="0 0.6 -0.4"/>
-  </xacro:default_camera>
-    <!-- Forward-looking sonar sensor  -->
-  <xacro:forward_multibeam_p900 namespace="${namespace}" parent_link="${namespace}/base_link">
-    <origin xyz="1.4 0 0.65" rpy="0 0 0"/>
-  </xacro:forward_multibeam_p900> -->
   <!-- Mount a GPS. -->
   <xacro:default_gps namespace="${namespace}" parent_link="${namespace}/base_link" />

File: uuv_sensor_plugins/uuv_sensor_ros_plugins/urdf/dvl_snippets.xacro (robot description, xacro)
@@ -1,3 +1,3 @@
-<?xml version="1.0"?>
+<?xml version="1.6"?>
 <!-- Copyright (c) 2020 The Plankton Authors.
      All rights reserved.

File: uuv_sensor_plugins/uuv_sensor_ros_plugins/urdf/sonar_snippets.xacro (robot description, xacro)
@@ -18,198 +18,146 @@
 -->
 <robot xmlns:xacro="http://www.ros.org/wiki/xacro">
-  <!-- Macro for a minimal collision block (for when you do not want collision block but gazebo needs one) -->
   <xacro:macro name="no_collision">
     <collision>
       <geometry>
-        <cylinder length="${0.000001}" radius="${0.000001}" />
+        <cylinder length="${0.1}" radius="${0.04}" />
       </geometry>
-      <origin xyz="0 0 0" rpy="0 ${0.5*pi} 0"/>
+      <origin xyz="0 0 0" rpy="0 0 0"/>
     </collision>
   </xacro:macro>
-  <!-- Side scan sonar -->
-  <xacro:macro name="sidescan_sonar" params="namespace parent_link suffix *origin">
-    <xacro:multibeam_sonar
+  <xacro:macro name="default_sonar_macro" params="namespace parent_link *origin inertial_reference_frame">
+    <xacro:sonar_plugin_macro
       namespace="${namespace}"
-      suffix="${suffix}"
       parent_link="${parent_link}"
-      topic="sss_${suffix}"
-      mass="0.015"
-      update_rate="2"
-      samples="60"
-      fov="${pi/3.0}"
-      range_min="1.0"
-      range_max="200.0"
-      range_stddev="0.027"
-      mesh="">
-      <inertia ixx="0.00001" ixy="0.0" ixz="0.0" iyy="0.00001" iyz="0.0" izz="0.00001" />
+      reference_frame="${inertial_reference_frame}"
+      update_rate="15"
+      topic="sonar"
+      noise_sigma="0.01"
+      noise_amplitude="0"
+      scale="1.0">
       <xacro:insert_block name="origin" />
-      <visual>
-        <origin xyz="0 0 0" rpy="0 0 0"/>
-        <geometry>
-          <box size="0.001 0.001 0.001"/>
-        </geometry>
-      </visual>
-    </xacro:multibeam_sonar>
+    </xacro:sonar_plugin_macro>
   </xacro:macro>
-  <!-- Inspired by m450-130: http://www.blueview.com/products/2d-imaging-sonar/m900-series/ -->
-  <xacro:macro name="forward_multibeam_sonar_m450_130" params="namespace parent_link *origin">
-    <xacro:multibeam_sonar
-      namespace="${namespace}"
-      suffix=""
-      parent_link="${parent_link}"
-      topic="sonar"
-      mass="2.015"
-      update_rate="25"
-      samples="768"
-      fov="2.27"
-      range_min="1.0"
-      range_max="100.0"
-      range_stddev="0.027"
-      mesh="">
-      <inertia ixx="0.00001" ixy="0.0" ixz="0.0" iyy="0.00001" iyz="0.0" izz="0.00001" />
-      <xacro:insert_block name="origin" />
-      <visual>
-        <geometry>
-          <mesh filename="file://$(find uuv_sensor_ros_plugins)/meshes/m450-130.dae" scale="1 1 1"/>
-        </geometry>
-      </visual>
-    </xacro:multibeam_sonar>
-  </xacro:macro>
-  <xacro:macro name="forward_multibeam_p900" params="namespace parent_link *origin">
-    <xacro:multibeam_sonar
-      namespace="${namespace}"
-      suffix=""
-      parent_link="${parent_link}"
-      topic="sonar"
-      mass="0.02"
-      update_rate="15"
-      samples="512"
-      fov="1.5708"
-      range_min="1.0"
-      range_max="100.0"
-      range_stddev="0.027"
-      mesh="">
-      <inertia ixx="0.00001" ixy="0.0" ixz="0.0" iyy="0.00001" iyz="0.0" izz="0.00001" />
-      <xacro:insert_block name="origin" />
-      <visual>
-        <geometry>
-          <mesh filename="file://$(find uuv_sensor_ros_plugins)/meshes/pingsonar.dae" scale="1 1 1"/>
-        </geometry>
-      </visual>
-    </xacro:multibeam_sonar>
-  </xacro:macro>
-  <xacro:macro name="multibeam_sonar"
-    params="namespace suffix parent_link topic mass update_rate
-      samples fov range_min range_max range_stddev mesh
-      *inertia *origin *visual">
-    <!-- Sensor link -->
-    <link name="${namespace}/sonar${suffix}_link">
+  <xacro:macro name="sonar_beam" params="namespace  pitch yaw update_rate">
+    <link name="${namespace}/sonar_beam_link">
+      <pose>0 0 0 0 0 0</pose>
       <inertial>
-        <xacro:insert_block name="inertia" />
-        <mass value="${mass}" />
+        <mass value="0.001" />  <!-- [kg] -->
         <origin xyz="0 0 0" rpy="0 0 0" />
+        <inertia ixx="0.000090623" ixy="0" ixz="0" iyy="0.000090623" iyz="0" izz="0.000091036" />
       </inertial>
-      <xacro:insert_block name="visual" />
       <xacro:no_collision/>
     </link>
-  <joint name="${namespace}_sonar${suffix}_joint" type="revolute">
-    <xacro:insert_block name="origin" />
-    <parent link="${parent_link}" />
-    <child link="${namespace}/sonar${suffix}_link" />
-    <limit upper="0" lower="0" effort="0" velocity="0" />
-    <axis xyz="1 0 0"/>
-  </joint>
-  <gazebo reference="${namespace}/sonar${suffix}_link">
-    <sensor type="gpu_ray" name="sonar${suffix}">
-      <pose>0 0 0 0 0 0</pose>
-      <visualize>false</visualize>
-      <update_rate>${update_rate}</update_rate>
-      <ray>
-        <scan>
-          <horizontal>
-            <samples>${samples}</samples>
-            <resolution>1</resolution>
-            <min_angle>-${0.5*fov}</min_angle>
-            <max_angle>${0.5*fov}</max_angle>
-          </horizontal>
-        </scan>
-        <range>
-          <min>${range_min}</min>
-          <max>${range_max}</max>
-          <resolution>0.01</resolution>
-        </range>
-        <noise>
-          <type>gaussian</type>
-          <mean>0.0</mean>
-          <stddev>${range_stddev}</stddev>
-        </noise>
-      </ray>
-      <plugin name="sonar${suffix}_controller" filename="libgazebo_ros_gpu_laser.so">
-        <topicName>${topic}</topicName>
-        <frameName>sonar${suffix}_link</frameName>
-      </plugin>
-      <!-- TODO: Separate switchable sonar version in another macro -->
-      <!-- <plugin name="switchable_sonar{suffix}_ros_interface" filename="libuuv_gazebo_ros_switchable_gpu_ray_sensor.so">
-          <namespace>${namespace}</namespace>
-          <input_topic>${topic}</input_topic>
-      </plugin> -->
-    </sensor>
-  </gazebo>
+    <joint name= "${namespace}/sonar_beam_joint" type="revolute">
+      <parent link="${namespace}/sonar_link" />
+      <child link="${namespace}/sonar_beam_link" />
+      <axis xyz="0 0 1"/>
+      <origin xyz="0 0 0.0"/>
+      <limit effort="5" lower="-10000000000000000" upper="10000000000000000" velocity="10.0"/>
+    </joint>
+    <gazebo reference="${namespace}/sonar_beam_link">
+      <sensor type="ray" name="sonar_ray">
+        <pose>0 0 0 0 0 0</pose>
+        <update_rate>${update_rate}</update_rate>
+        <visualize>true</visualize>
+        <ray>
+          <scan>
+            <horizontal>
+              <samples>3</samples>
+              <resolution>1</resolution>
+              <min_angle>-0.034906585</min_angle>
+              <max_angle>0.034906585</max_angle>
+            </horizontal>
+            <vertical>
+              <samples>50</samples>
+              <resolution>1</resolution>
+              <min_angle>-0.4363</min_angle>
+              <max_angle>0.4363</max_angle>
+            </vertical>
+          </scan>
+          <range>
+            <min>0.75</min>
+            <max>50</max>
+            <resolution>0.08</resolution>
+          </range>
+          <noise>
+            <type>gaussian</type>
+            <mean>0.0</mean>
+            <stddev>0.005</stddev>
+          </noise>
+        </ray>
+        <plugin filename="libgazebo_ros_ray_sensor.so" name="sonar_beam">
+          <ros>
+            <remapping>~/out:=${topic}/range</remapping>
+          </ros>
+          <!-- <gaussianNoise>0.005</gaussianNoise> -->
+          <alwaysOn>true</alwaysOn>
+          <!-- <updateRate>${update_rate}</updateRate> -->
+          <!-- <topicName>${topic}_sonar${index}</topicName> -->
+          <frame_name>${namespace}/sonar_link</frame_name>
+          <!-- TODO Check for fov -->
+          <!-- <fov>0.06</fov> -->
+          <radiation_type>ultrasound</radiation_type>
+          <!-- Set output to sensor_msgs/Range to get same output type as gazebo_ros_range -->
+          <output_type>sensor_msgs/Range</output_type>
+        </plugin>
+        <plugin filename="libgazebo_ros_ray_sensor.so" name="sonar_PointCloud2">
+          <ros>
+            <remapping>~/out:=${topic}/PointCloud2</remapping>
+          </ros>
+          <!-- <gaussianNoise>0.005</gaussianNoise> -->
+          <alwaysOn>true</alwaysOn>
+          <!-- <updateRate>${update_rate}</updateRate> -->
+          <!-- <topicName>${topic}_sonar${index}</topicName> -->
+          <frame_name>${namespace}/sonar_link</frame_name>
+          <!-- TODO Check for fov -->
+          <!-- <fov>0.06</fov> -->
+          <radiation_type>ultrasound</radiation_type>
+          <!-- Set output to sensor_msgs/Range to get same output type as gazebo_ros_range -->
+          <output_type>sensor_msgs/PointCloud2</output_type>
+        </plugin>
+      </sensor>
+    </gazebo>
   </xacro:macro>
-  <xacro:macro name="forward_looking_sonar"
-    params="namespace suffix parent_link topic mass update_rate
-      samples fov width height *inertia *origin">
-    <!-- Sensor link -->
-    <link name="${namespace}/forward_sonar${suffix}_link">
+  <xacro:macro name="sonar_plugin_macro"
+    params="namespace  parent_link topic scale *origin update_rate
+    reference_frame noise_sigma noise_amplitude">
+    <link name="${namespace}/sonar_link">
+      <pose>0 0 0.0 0 0 0</pose>
       <inertial>
-        <xacro:insert_block name="inertia" />
-        <mass value="${mass}" />
+        <mass value="0.51" />  <!-- [kg] -->
         <origin xyz="0 0 0" rpy="0 0 0" />
+        <inertia ixx="0.00055" ixy="0" ixz="0" iyy="0.00055" iyz="0" izz="0.00170" />
       </inertial>
       <visual>
         <geometry>
-          <mesh filename="file://$(find uuv_sensor_ros_plugins)/meshes/oe14-372.dae" scale="1 1 1"/>
+          <mesh filename="file://$(find uuv_sensor_ros_plugins)/meshes/pingsonar.dae" scale="${scale} ${scale} ${scale}"/>
         </geometry>
       </visual>
       <xacro:no_collision/>
     </link>
-    <joint name="${namespace}_forward_sonar${suffix}_joint" type="revolute">
+    <joint name="${namespace}/sonar_joint" type="revolute">
       <xacro:insert_block name="origin" />
       <parent link="${parent_link}" />
-      <child link="${namespace}/forward_sonar${suffix}_link" />
+      <child link="${namespace}/sonar_link" />
       <limit upper="0" lower="0" effort="0" velocity="0" />
       <axis xyz="1 0 0"/>
     </joint>
-    <gazebo reference="${namespace}/forward_sonar${suffix}_link">
-      <sensor name="${namespace}/image_sonar" type="depth">
-        <camera>
-          <horizontal_fov>${fov}</horizontal_fov>
-              <image>
-                <width>${width}</width>
-                <height>${height}</height>
-                <format>R8G8B8</format>
-              </image>
-              <clip>
-                <near>0.1</near>
-                <far>17</far>
-              </clip>
-              <save enabled="true">
-                <path>/tmp/camera</path>
-              </save>
-        </camera>
-        <plugin filename="libimage_sonar_ros_plugin.so" name="forward_sonar${suffix}_controller">
-          <topicName>${topic}</topicName>
-            <frameName>forward_sonar${suffix}_optical_frame</frameName>
-        </plugin>
-        <always_on>true</always_on>
-	      <update_rate>${update_rate}</update_rate>
-      </sensor>
+    <xacro:sonar_beam
+      namespace="${namespace}"
+      pitch="0.0" yaw="0.0" update_rate="${update_rate}">
+    </xacro:sonar_beam>
+    <gazebo>
+      <plugin filename="libuuv_gazebo_ros_sonar_plugin.so" name="libuuv_gazebo_ros_sonar_plugin">
+        <!-- <updateRate>${update_rate}</updateRate> -->
+        <!-- <topicName>${topic}_sonar${index}</topicName> -->
+        <velocity>10.0</velocity>
+        <!-- <robot_namespace>${namespace}</robot_namespace> -->
+        <link_name>${namespace}/sonar_link</link_name> <!-- (string, required): name of the body which holds the IMU sensor -->
+        <sensor_topic>${topic}</sensor_topic> <!-- (string): name of the sensor output topic and prefix of service names (defaults to imu) -->
+        <update_rate>${update_rate}</update_rate> <!-- Update period of accelerometer and gyroscope [s] -->
+        <enable_gazebo_messages>false</enable_gazebo_messages>
+      </plugin>
     </gazebo>
-	<joint name="${namespace}/forward_sonar${suffix}_joint" type="fixed">
-      <origin xyz="0 0 0" rpy="${-pi/2} 0 ${-pi/2}"/>
-      <parent link="${namespace}/forward_sonar${suffix}_link"/>
-      <child link="${namespace}/forward_sonar${suffix}_optical_frame"/>
-    </joint>
-	<link name="${namespace}/forward_sonar${suffix}_optical_frame"/>
   </xacro:macro>
 </robot>
