Commit message: Simulator updates

File: uuv_sensor_plugins/uuv_sensor_ros_plugins/urdf/stereo_snippets.xacro (robot description, xacro)
@@ -18,15 +18,4 @@
 -->
 <robot xmlns:xacro="http://www.ros.org/wiki/xacro">
-  <xacro:property name="k1l" value="-0.389021"/>
-  <xacro:property name="k2l" value="0.118184"/>
-  <xacro:property name="p1l" value="0.001259"/>
-  <xacro:property name="p2l" value="0.002050"/>
-  <xacro:property name="k3l" value="0.000000"/>
-  <xacro:property name="k1r" value="-0.378206"/>
-  <xacro:property name="k2r" value="0.104833"/>
-  <xacro:property name="p1r" value="0.000458"/>
-  <xacro:property name="p2r" value="0.002447"/>
-  <xacro:property name="k3r" value="0.000000"/>
-  <xacro:property name="hfov" value="1.3844"/>
   <!-- Macro for a minimal collision block (for when you do not want collision block but gazebo needs one) -->
   <xacro:macro name="no_collision">
@@ -38,122 +27,156 @@
     </collision>
   </xacro:macro>
-  <xacro:macro name="duo3d_camera" params="namespace parent_link *origin">
-    <link name="${namespace}/duo3d_left_link">
+  <xacro:macro name="zed2_macro" params="namespace parent_link  *origin">
+    <xacro:zed2_camera_plugin
+      namespace="${namespace}"
+      parent_link="${parent_link}"
+      topic="camera"
+      mass="0.015"
+      update_rate="30"
+      hfov="1.8125"
+      width="768"
+      height="492"
+      stddev="0.02"
+      scale="1.0">
+      <inertia ixx="0.00001" ixy="0.0" ixz="0.0" iyy="0.00001" iyz="0.0" izz="0.00001" />
+      <xacro:insert_block name="origin" />>
+    </xacro:zed2_camera_plugin>
+  </xacro:macro>
+  <xacro:macro name="zed2_camera_plugin"
+    params="namespace  parent_link topic mass update_rate
+      hfov width height stddev scale
+      *inertia *origin">
+    <!-- Sensor link -->
+    <link name="${namespace}/camera_link">
       <inertial>
-        <mass value="0.01"/>
-        <inertia ixx="0" ixy="0.0" ixz="0.0" iyy="0" iyz="0.0" izz="0" />
+        <xacro:insert_block name="inertia" />
+        <mass value="${mass}" />
+        <origin xyz="0 0 0" rpy="0 0 0" />
       </inertial>
       <visual>
         <geometry>
-          <mesh filename="file://$(find uuv_sensor_ros_plugins)/meshes/duo3d.dae"/>
+          <mesh filename="file://$(find uuv_sensor_ros_plugins)/meshes/zed2.stl" scale="${scale} ${scale} ${scale}"/>
         </geometry>
       </visual>
       <xacro:no_collision/>
     </link>
-    <joint name="${namespace}/duo3d_joint" type="revolute">
+    <joint name="${namespace}/camera_joint" type="revolute">
       <xacro:insert_block name="origin" />
       <parent link="${parent_link}" />
-      <child link="${namespace}/duo3d_left_link" />
+      <child link="${namespace}/camera_link" />
       <limit upper="0" lower="0" effort="0" velocity="0" />
       <axis xyz="1 0 0"/>
     </joint>
-    <gazebo reference="${namespace}/duo3d_left_link">
-      <sensor name="camera" type="camera">
-      <camera>
-        <horizontal_fov>${hfov}</horizontal_fov>
-        <image>
-          <width>640</width>
-          <height>460</height>
-          <format>R8G8B8</format>
-        </image>
-        <clip>
-          <near>0.05</near>
-          <far>5000</far>
-        </clip>
-        <distortion>
-          <k1>${k1l}</k1>
-          <k2>${k2l}</k2>
-          <k3>${k3l}</k3>
-          <p1>${p1l}</p1>
-          <p2>${p2l}</p2>
-          <center>0.5 0.5</center>
-        </distortion>
-      </camera>
-      <plugin name="left_controller" filename="libgazebo_ros_camera.so">
-        <ros>
-          <remapping>image_raw:=image_raw</remapping>
-          <remapping>camera_info:=camera_info</remapping>
-        </ros>
-        <!-- <alwaysOn>true</alwaysOn> -->
-        <!-- <updateRate>30.0</updateRate> -->
-        <camera_name>${namespace}/duo3d_left</camera_name>
-        <!-- <cameraName>${namespace}/duo3d_left</cameraName> -->
-        <!-- <imageTopicName>image_raw</imageTopicName> -->
-        <!-- <cameraInfoTopicName>camera_info</cameraInfoTopicName> -->
-        <frame_name>${namespace}/duo3d_left_link</frame_name>
-        <!-- <frameName>${namespace}/duo3d_left_link</frameName> -->
-         <hack_baseline>0.07</hack_baseline>
-        <!-- <hackBaseline>0.07</hackBaseline> -->
-        <!-- <distortionK1>${k1l}</distortionK1>
-        <distortionK2>${k2l}</distortionK2>
-        <distortionK3>${k3l}</distortionK3>
-        <distortionT1>${p1l}</distortionT1>
-        <distortionT2>${p2l}</distortionT2> -->
-      </plugin>
-      <always_on>1</always_on>
-      <update_rate>30</update_rate>
-      <visualize>true</visualize>
-    </sensor>
-    </gazebo>
-    <link name="${namespace}/duo3d_right_link">
-      <inertial>
-        <mass value="0.01"/>
-        <inertia ixx="0" ixy="0.0" ixz="0.0" iyy="0" iyz="0.0" izz="0" />
-      </inertial>
-      <xacro:no_collision/>
+    <link name="${namespace}/camera_link_optical">
+      <xacro:box_inertial x="0.0001" y="0.0001" z="0.0001" mass="0.001">
+        <origin xyz="0 0 0" rpy="0 0 0"/>
+      </xacro:box_inertial>
+      <collision>
+        <!-- todo: gazebo needs a collision volume or it will ignore the pose of
+           the joint that leads to this link (and assume it to be the identity) -->
+        <geometry>
+          <cylinder length="0.000001" radius="0.000001"/>
+        </geometry>
+        <origin xyz="0 0 0" rpy="0 ${0.5*pi} 0"/>
+      </collision>
     </link>
-    <joint name="${namespace}/duo3d_right_joint" type="revolute">
-      <origin xyz="0.0 -0.03 0" rpy="0 0 0"/>
-      <parent link="${namespace}/duo3d_left_link" />
-      <child link="${namespace}/duo3d_right_link" />
+    <joint name="${namespace}/camera_optical_joint" type="revolute">
+      <origin xyz="0 0 0" rpy="${-pi/2} 0 ${-pi/2}"/>
+      <parent link="${namespace}/camera_link"/>
+      <child link="${namespace}/camera_link_optical"/>
       <limit upper="0" lower="0" effort="0" velocity="0" />
       <axis xyz="1 0 0"/>
     </joint>
-    <gazebo reference="${namespace}/duo3d_right_link">
-      <sensor name="camera" type="camera">
-      <camera>
-        <horizontal_fov>${hfov}</horizontal_fov>
-        <image>
-          <width>640</width>
-          <height>460</height>
-          <format>R8G8B8</format>
-        </image>
-        <clip>
-          <near>0.05</near>
-          <far>5000</far>
-        </clip>
-        <distortion>
-          <k1>${k1l}</k1>
-          <k2>${k2l}</k2>
-          <k3>${k3l}</k3>
-          <p1>${p1l}</p1>
-          <p2>${p2l}</p2>
-          <center>0.5 0.5</center>
-        </distortion>
-      </camera>
-      <plugin name="right_controller" filename="libgazebo_ros_camera.so">
-        <ros>
-          <remapping>image_raw:=image_raw</remapping>
-          <remapping>camera_info:=camera_info</remapping>
-        </ros>
-        <camera_name>${namespace}/duo3d_right</camera_name>
-        <frame_name>${namespace}/duo3d_right_link</frame_name>
-        <hack_baseline>0.07</hack_baseline>
-      </plugin>
-      <always_on>1</always_on>
-      <update_rate>30</update_rate>
-      <visualize>true</visualize>
-    </sensor>
-  </gazebo>
+    <gazebo reference="${namespace}/camera_link">
+      <sensor type="depth" name="zed2_depth">
+        <update_rate>${update_rate}</update_rate>
+        <visualize>false</visualize>
+        <camera name="depth_camera">
+          <horizontal_fov>${hfov}</horizontal_fov>
+          <image>
+            <width>${width}</width>
+            <height>${height}</height>
+            <format>R8G8B8</format>
+          </image>
+          <depth_camera>
+          </depth_camera>
+          <clip>
+            <near>0.02</near>
+            <far>300</far>
+          </clip>
+          <noise>
+            <type>gaussian</type>
+            <mean>0.0</mean>
+            <stddev>${stddev}</stddev>
+          </noise>
+        </camera>
+        <plugin name="camera_controller" filename="libgazebo_ros_camera.so">
+          <!-- <updateRate>${update_rate}</updateRate> -->
+          <camera_name>${namespace}/camera</camera_name>
+          <!-- <cameraName>${namespace}/camera${suffix}</cameraName> -->
+          <frame_name>camera_link_optical</frame_name>
+          <!-- <frameName>camera${suffix}_link_optical</frameName> -->
+          <attenuationR>0.0</attenuationR>
+          <attenuationG>0.0</attenuationG>
+          <attenuationB>0.0</attenuationB>
+          <backgroundR>0</backgroundR>
+          <backgroundG>0</backgroundG>
+          <backgroundB>0</backgroundB>
+          <ros>
+            <!-- Use either <argument> with - -ros-args -r or remapping -->
+            <namespace>{namespace}</namespace>
+            <remapping>image_raw:=${topic}_image</remapping>
+            <remapping>${namespace}/camera/image_raw:=zed2/image_demo</remapping>
+            <remapping>${namespace}/camera/depth/image_raw:=zed2/depth_demo</remapping>
+            <remapping>${namespace}/camera/camera_info:=zed2/raw_cam_info_demo</remapping>
+            <remapping>${namespace}/camera/depth/camera_info:=zed2/depth_cam_info_demo</remapping>
+            <remapping>${namespace}/camera/points:=zed2/points_demo</remapping>
+          </ros>
+          <!-- Only useful for depth camera -->
+          <!-- <min_depth>10.0</min_depth> -->
+          <!-- required for ros depth cam -->
+          <!-- <imageTopicName>${topic}_image</imageTopicName> -->
+          <!-- TODO why depth info were here ? -->
+          <!-- <pointCloudTopicName>${topic}_cloud</pointCloudTopicName>
+          <depthImageTopicName>${topic}_depth</depthImageTopicName>
+          <depthImageCameraInfoTopicName>${topic}_depth_info</depthImageCameraInfoTopicName> -->
+          <!-- <pointCloudCutoff>10.0</pointCloudCutoff> -->
+        </plugin>
+      </sensor>
+      <sensor type="camera" name="zed_rgb">
+        <update_rate>60</update_rate>
+        <visualize>false</visualize>
+        <camera name="rgb_camera">
+          <horizontal_fov>1.3962634</horizontal_fov>
+          <image>
+            <width>640</width>
+            <height>480</height>
+            <format>R8G8B8</format>
+          </image>
+          <clip>
+            <near>0.02</near>
+            <far>300</far>
+          </clip>
+          <noise>
+            <type>gaussian</type>
+            <!-- Noise is sampled independently per pixel on each frame.
+                 That pixel's noise value is added to each of its color
+                 channels, which at that point lie in the range [0,1]. -->
+            <mean>0.0</mean>
+            <stddev>0.007</stddev>
+          </noise>
+        </camera>
+        <plugin name="camera_controller" filename="libgazebo_ros_camera.so">
+          <ros>
+            <namespace>{namespace}</namespace>
+            <!-- TODO(louise) Remapping not working due to https://github.com/ros-perception/image_common/issues/93 -->
+            <remapping>image_raw:=zed2/rgb_image_demo</remapping>
+            <remapping>camera_info:=zed2/rgb_camera_info_demo</remapping>
+          </ros>
+          <!-- camera_name>omit so it defaults to sensor name</camera_name-->
+          <!-- frame_name>omit so it defaults to link name</frame_name-->
+        </plugin>
+      </sensor>
+    </gazebo>
   </xacro:macro>
 </robot>
